File: ATMEGAx4SeriesCoprocessor.sch (KiCad schematic (older format))
At the start: 7 parts, among them J12 Conn_01x03, J13 AVR-ISP-6, J14 Conn_01x06 (Serial Connector), U18 ATmega1284P-PU

Commit message: Keep futzing with the design
Added a missing +5v power source to the x4 coprocessor schematic
Connections:
- net +5V: now also C27.1, U18.30 (AVCC)
Changed lines of the file:
@@
 P 3400 3250
 AR Path="/7D8CCC7A/7D8FC773" Ref="U18"  Part="1"
-AR Path="/847B579A/7D8FC773" Ref="U?"  Part="1"
-F 0 "U?" H 3400 1161 50  0000 C CNN
+AR Path="/847B579A/7D8FC773" Ref="U19"  Part="1"
+F 0 "U18" H 3400 1161 50  0000 C CNN
 F 1 "ATmega1284P-PU" H 3400 1070 50  0000 C CNN
 F 2 "Package_DIP:DIP-40_W15.24mm_Socket" H 3400 3250 50  0001 C CIN
@@
 P 3400 850
 AR Path="/7D8CCC7A/7D8FC77F" Ref="#PWR066"  Part="1"
-AR Path="/847B579A/7D8FC77F" Ref="#PWR?"  Part="1"
-F 0 "#PWR?" H 3400 700 50  0001 C CNN
+AR Path="/847B579A/7D8FC77F" Ref="#PWR0103"  Part="1"
+F 0 "#PWR0103" H 3400 700 50  0001 C CNN
 F 1 "+5V" H 3415 1023 50  0000 C CNN
 F 2 "" H 3400 850 50  0001 C CNN
@@
 P 3400 5750
 AR Path="/7D8CCC7A/7D8FC785" Ref="#PWR067"  Part="1"
-AR Path="/847B579A/7D8FC785" Ref="#PWR?"  Part="1"
-F 0 "#PWR?" H 3400 5500 50  0001 C CNN
+AR Path="/847B579A/7D8FC785" Ref="#PWR0104"  Part="1"
+F 0 "#PWR0104" H 3400 5500 50  0001 C CNN
 F 1 "GND" H 3405 5577 50  0000 C CNN
 F 2 "" H 3400 5750 50  0001 C CNN
@@
 P 2050 2550
 AR Path="/7D8CCC7A/7D8FC78C" Ref="C27"  Part="1"
-AR Path="/847B579A/7D8FC78C" Ref="C?"  Part="1"
-F 0 "C?" H 2165 2596 50  0000 L CNN
+AR Path="/847B579A/7D8FC78C" Ref="C30"  Part="1"
+F 0 "C27" H 2165 2596 50  0000 L CNN
 F 1 "0.1uF" H 2165 2505 50  0000 L CNN
 F 2 "Capacitor_SMD:C_0805_2012Metric_Pad1.18x1.45mm_HandSolder" H 2088 2400 50  0001 C CNN
@@
 P 2500 2900
 AR Path="/7D8CCC7A/7D8FC798" Ref="C28"  Part="1"
-AR Path="/847B579A/7D8FC798" Ref="C?"  Part="1"
-F 0 "C?" H 2615 2946 50  0000 L CNN
+AR Path="/847B579A/7D8FC798" Ref="C31"  Part="1"
+F 0 "C28" H 2615 2946 50  0000 L CNN
 F 1 "0.1uF" H 2615 2855 50  0000 L CNN
 F 2 "Capacitor_SMD:C_0805_2012Metric_Pad1.18x1.45mm_HandSolder" H 2538 2750 50  0001 C CNN
@@
 P 1450 2750
 AR Path="/7D8CCC7A/7D8FC79F" Ref="#PWR065"  Part="1"
-AR Path="/847B579A/7D8FC79F" Ref="#PWR?"  Part="1"
-F 0 "#PWR?" H 1450 2500 50  0001 C CNN
+AR Path="/847B579A/7D8FC79F" Ref="#PWR0105"  Part="1"
+F 0 "#PWR0105" H 1450 2500 50  0001 C CNN
 F 1 "GND" H 1455 2577 50  0000 C CNN
 F 2 "" H 1450 2750 50  0001 C CNN
@@
 P 9550 1600
 AR Path="/7D8CCC7A/65D0C082" Ref="J13"  Part="1"
-AR Path="/847B579A/65D0C082" Ref="J?"  Part="1"
-F 0 "J?" H 9221 1696 50  0000 R CNN
+AR Path="/847B579A/65D0C082" Ref="J23"  Part="1"
+F 0 "J13" H 9221 1696 50  0000 R CNN
 F 1 "AVR-ISP-6" H 9221 1605 50  0000 R CNN
 F 2 "Connector_PinHeader_2.54mm:PinHeader_2x03_P2.54mm_Vertical" V 9300 1650 50  0001 C CNN
@@
 P 9450 800
 AR Path="/7D8CCC7A/65D67928" Ref="#PWR068"  Part="1"
-AR Path="/847B579A/65D67928" Ref="#PWR?"  Part="1"
-F 0 "#PWR?" H 9450 650 50  0001 C CNN
+AR Path="/847B579A/65D67928" Ref="#PWR0106"  Part="1"
+F 0 "#PWR0106" H 9450 650 50  0001 C CNN
 F 1 "+5V" H 9465 973 50  0000 C CNN
 F 2 "" H 9450 800 50  0001 C CNN
@@
 P 9450 2400
 AR Path="/7D8CCC7A/65D7AB96" Ref="#PWR069"  Part="1"
-AR Path="/847B579A/65D7AB96" Ref="#PWR?"  Part="1"
-F 0 "#PWR?" H 9450 2150 50  0001 C CNN
+AR Path="/847B579A/65D7AB96" Ref="#PWR0107"  Part="1"
+F 0 "#PWR0107" H 9450 2150 50  0001 C CNN
 F 1 "GND" H 9455 2227 50  0000 C CNN
 F 2 "" H 9450 2400 50  0001 C CNN
@@
 P 9600 3450
 AR Path="/7D8CCC7A/623C8548" Ref="J14"  Part="1"
-AR Path="/847B579A/623C8548" Ref="J?"  Part="1"
-F 0 "J?" H 9518 2925 50  0000 C CNN
+AR Path="/847B579A/623C8548" Ref="J24"  Part="1"
+F 0 "J14" H 9518 2925 50  0000 C CNN
 F 1 "Conn_01x06 (Serial Connector)" H 9518 3016 50  0000 C CNN
 F 2 "Connector_PinHeader_2.54mm:PinHeader_1x06_P2.54mm_Vertical" H 9600 3450 50  0001 C CNN
@@
 P 10100 2750
 AR Path="/7D8CCC7A/65E08A07" Ref="#PWR070"  Part="1"
-AR Path="/847B579A/65E08A07" Ref="#PWR?"  Part="1"
-F 0 "#PWR?" H 10100 2600 50  0001 C CNN
+AR Path="/847B579A/65E08A07" Ref="#PWR0108"  Part="1"
+F 0 "#PWR0108" H 10100 2600 50  0001 C CNN
 F 1 "+5V" H 10115 2923 50  0000 C CNN
 F 2 "" H 10100 2750 50  0001 C CNN
@@
 P 10350 4400
 AR Path="/7D8CCC7A/65DF3F8A" Ref="#PWR071"  Part="1"
-AR Path="/847B579A/65DF3F8A" Ref="#PWR?"  Part="1"
-F 0 "#PWR?" H 10350 4150 50  0001 C CNN
+AR Path="/847B579A/65DF3F8A" Ref="#PWR0109"  Part="1"
+F 0 "#PWR0109" H 10350 4150 50  0001 C CNN
 F 1 "GND" H 10355 4227 50  0000 C CNN
 F 2 "" H 10350 4400 50  0001 C CNN
@@
 P 9650 4250
 AR Path="/7D8CCC7A/65D916C2" Ref="C29"  Part="1"
-AR Path="/847B579A/65D916C2" Ref="C?"  Part="1"
-F 0 "C?" V 9398 4250 50  0000 C CNN
+AR Path="/847B579A/65D916C2" Ref="C32"  Part="1"
+F 0 "C29" V 9398 4250 50  0000 C CNN
 F 1 "0.1uF" V 9489 4250 50  0000 C CNN
 F 2 "Capacitor_SMD:C_0805_2012Metric_Pad1.18x1.45mm_HandSolder" H 9688 4100 50  0001 C CNN
@@
 P 7350 5900
 AR Path="/7D8CCC7A/7DB0C2C2" Ref="J12"  Part="1"
-AR Path="/847B579A/7DB0C2C2" Ref="J?"  Part="1"
-F 0 "J?" H 7430 5942 50  0000 L CNN
+AR Path="/847B579A/7DB0C2C2" Ref="J22"  Part="1"
+F 0 "J12" H 7430 5942 50  0000 L CNN
 F 1 "Conn_01x03" H 7430 5851 50  0000 L CNN
 F 2 "Connector_PinHeader_2.54mm:PinHeader_1x03_P2.54mm_Vertical" H 7350 5900 50  0001 C CNN
@@
 Text HLabel 5800 1550 2    50   UnSpc ~ 0
 PA0
+$Comp
+L power:+5V #PWR0110
+U 1 1 8791B6EA
+P 3500 600
+AR Path="/7D8CCC7A/8791B6EA" Ref="#PWR0110"  Part="1"
+AR Path="/847B579A/8791B6EA" Ref="#PWR0111"  Part="1"
+F 0 "#PWR0111" H 3500 450 50  0001 C CNN
+F 1 "+5V" H 3515 773 50  0000 C CNN
+F 2 "" H 3500 600 50  0001 C CNN
+F 3 "" H 3500 600 50  0001 C CNN
+	1    3500 600
+	1    0    0    -1
+$EndComp
+Connection ~ 3500 600
 $EndSCHEMATC

Commit message: Finish cleaning up rev3 for now the layout is complete
Changed lines of the file:
@@
 AR Path="/7D8CCC7A/7D8FC773" Ref="U18"  Part="1"
 AR Path="/847B579A/7D8FC773" Ref="U19"  Part="1"
-F 0 "U18" H 3400 1161 50  0000 C CNN
+F 0 "U19" H 3400 1161 50  0000 C CNN
 F 1 "ATmega1284P-PU" H 3400 1070 50  0000 C CNN
 F 2 "Package_DIP:DIP-40_W15.24mm_Socket" H 3400 3250 50  0001 C CIN
@@
 AR Path="/7D8CCC7A/7D8FC77F" Ref="#PWR066"  Part="1"
 AR Path="/847B579A/7D8FC77F" Ref="#PWR0103"  Part="1"
-F 0 "#PWR066" H 3400 700 50  0001 C CNN
+F 0 "#PWR0103" H 3400 700 50  0001 C CNN
 F 1 "+5V" H 3415 1023 50  0000 C CNN
 F 2 "" H 3400 850 50  0001 C CNN
@@
 AR Path="/7D8CCC7A/7D8FC785" Ref="#PWR067"  Part="1"
 AR Path="/847B579A/7D8FC785" Ref="#PWR0104"  Part="1"
-F 0 "#PWR067" H 3400 5500 50  0001 C CNN
+F 0 "#PWR0104" H 3400 5500 50  0001 C CNN
 F 1 "GND" H 3405 5577 50  0000 C CNN
 F 2 "" H 3400 5750 50  0001 C CNN
@@
 AR Path="/7D8CCC7A/7D8FC78C" Ref="C27"  Part="1"
 AR Path="/847B579A/7D8FC78C" Ref="C30"  Part="1"
-F 0 "C27" H 2165 2596 50  0000 L CNN
+F 0 "C30" H 2165 2596 50  0000 L CNN
 F 1 "0.1uF" H 2165 2505 50  0000 L CNN
 F 2 "Capacitor_SMD:C_0805_2012Metric_Pad1.18x1.45mm_HandSolder" H 2088 2400 50  0001 C CNN
@@
 AR Path="/7D8CCC7A/7D8FC798" Ref="C28"  Part="1"
 AR Path="/847B579A/7D8FC798" Ref="C31"  Part="1"
-F 0 "C28" H 2615 2946 50  0000 L CNN
+F 0 "C31" H 2615 2946 50  0000 L CNN
 F 1 "0.1uF" H 2615 2855 50  0000 L CNN
 F 2 "Capacitor_SMD:C_0805_2012Metric_Pad1.18x1.45mm_HandSolder" H 2538 2750 50  0001 C CNN
@@
 AR Path="/7D8CCC7A/7D8FC79F" Ref="#PWR065"  Part="1"
 AR Path="/847B579A/7D8FC79F" Ref="#PWR0105"  Part="1"
-F 0 "#PWR065" H 1450 2500 50  0001 C CNN
+F 0 "#PWR0105" H 1450 2500 50  0001 C CNN
 F 1 "GND" H 1455 2577 50  0000 C CNN
 F 2 "" H 1450 2750 50  0001 C CNN
@@
 AR Path="/7D8CCC7A/65D0C082" Ref="J13"  Part="1"
 AR Path="/847B579A/65D0C082" Ref="J23"  Part="1"
-F 0 "J13" H 9221 1696 50  0000 R CNN
+F 0 "J23" H 9221 1696 50  0000 R CNN
 F 1 "AVR-ISP-6" H 9221 1605 50  0000 R CNN
 F 2 "Connector_PinHeader_2.54mm:PinHeader_2x03_P2.54mm_Vertical" V 9300 1650 50  0001 C CNN
@@
 AR Path="/7D8CCC7A/65D67928" Ref="#PWR068"  Part="1"
 AR Path="/847B579A/65D67928" Ref="#PWR0106"  Part="1"
-F 0 "#PWR068" H 9450 650 50  0001 C CNN
+F 0 "#PWR0106" H 9450 650 50  0001 C CNN
 F 1 "+5V" H 9465 973 50  0000 C CNN
 F 2 "" H 9450 800 50  0001 C CNN
@@
 AR Path="/7D8CCC7A/65D7AB96" Ref="#PWR069"  Part="1"
 AR Path="/847B579A/65D7AB96" Ref="#PWR0107"  Part="1"
-F 0 "#PWR069" H 9450 2150 50  0001 C CNN
+F 0 "#PWR0107" H 9450 2150 50  0001 C CNN
 F 1 "GND" H 9455 2227 50  0000 C CNN
 F 2 "" H 9450 2400 50  0001 C CNN
@@
 AR Path="/7D8CCC7A/623C8548" Ref="J14"  Part="1"
 AR Path="/847B579A/623C8548" Ref="J24"  Part="1"
-F 0 "J14" H 9518 2925 50  0000 C CNN
+F 0 "J24" H 9518 2925 50  0000 C CNN
 F 1 "Conn_01x06 (Serial Connector)" H 9518 3016 50  0000 C CNN
 F 2 "Connector_PinHeader_2.54mm:PinHeader_1x06_P2.54mm_Vertical" H 9600 3450 50  0001 C CNN
@@
 AR Path="/7D8CCC7A/65E08A07" Ref="#PWR070"  Part="1"
 AR Path="/847B579A/65E08A07" Ref="#PWR0108"  Part="1"
-F 0 "#PWR070" H 10100 2600 50  0001 C CNN
+F 0 "#PWR0108" H 10100 2600 50  0001 C CNN
 F 1 "+5V" H 10115 2923 50  0000 C CNN
 F 2 "" H 10100 2750 50  0001 C CNN
@@
 AR Path="/7D8CCC7A/65DF3F8A" Ref="#PWR071"  Part="1"
 AR Path="/847B579A/65DF3F8A" Ref="#PWR0109"  Part="1"
-F 0 "#PWR071" H 10350 4150 50  0001 C CNN
+F 0 "#PWR0109" H 10350 4150 50  0001 C CNN
 F 1 "GND" H 10355 4227 50  0000 C CNN
 F 2 "" H 10350 4400 50  0001 C CNN
@@
 AR Path="/7D8CCC7A/65D916C2" Ref="C29"  Part="1"
 AR Path="/847B579A/65D916C2" Ref="C32"  Part="1"
-F 0 "C29" V 9398 4250 50  0000 C CNN
+F 0 "C32" V 9398 4250 50  0000 C CNN
 F 1 "0.1uF" V 9489 4250 50  0000 C CNN
 F 2 "Capacitor_SMD:C_0805_2012Metric_Pad1.18x1.45mm_HandSolder" H 9688 4100 50  0001 C CNN
@@
 AR Path="/7D8CCC7A/7DB0C2C2" Ref="J12"  Part="1"
 AR Path="/847B579A/7DB0C2C2" Ref="J22"  Part="1"
-F 0 "J12" H 7430 5942 50  0000 L CNN
+F 0 "J22" H 7430 5942 50  0000 L CNN
 F 1 "Conn_01x03" H 7430 5851 50  0000 L CNN
 F 2 "Connector_PinHeader_2.54mm:PinHeader_1x03_P2.54mm_Vertical" H 7350 5900 50  0001 C CNN
@@
 AR Path="/7D8CCC7A/8791B6EA" Ref="#PWR0110"  Part="1"
 AR Path="/847B579A/8791B6EA" Ref="#PWR0111"  Part="1"
-F 0 "#PWR0110" H 3500 450 50  0001 C CNN
+F 0 "#PWR0111" H 3500 450 50  0001 C CNN
 F 1 "+5V" H 3515 773 50  0000 C CNN
 F 2 "" H 3500 600 50  0001 C CNN

Commit message: Added a pullup resistor for each programming reset line
Parts:
- added R7: 10k, Resistor_SMD:R_0805_2012Metric_Pad1.20x1.40mm_HandSolder, symbol Device:R
Connections:
- net +5V: now also R7.1
- net ~PRG_RESET: now also R7.2
Changed lines of the file:
@@
 AR Path="/7D8CCC7A/7D8FC773" Ref="U18"  Part="1"
 AR Path="/847B579A/7D8FC773" Ref="U19"  Part="1"
-F 0 "U19" H 3400 1161 50  0000 C CNN
+F 0 "U18" H 3400 1161 50  0000 C CNN
 F 1 "ATmega1284P-PU" H 3400 1070 50  0000 C CNN
 F 2 "Package_DIP:DIP-40_W15.24mm_Socket" H 3400 3250 50  0001 C CIN
@@
 AR Path="/7D8CCC7A/7D8FC77F" Ref="#PWR066"  Part="1"
 AR Path="/847B579A/7D8FC77F" Ref="#PWR0103"  Part="1"
-F 0 "#PWR0103" H 3400 700 50  0001 C CNN
+F 0 "#PWR066" H 3400 700 50  0001 C CNN
 F 1 "+5V" H 3415 1023 50  0000 C CNN
 F 2 "" H 3400 850 50  0001 C CNN
@@
 AR Path="/7D8CCC7A/7D8FC785" Ref="#PWR067"  Part="1"
 AR Path="/847B579A/7D8FC785" Ref="#PWR0104"  Part="1"
-F 0 "#PWR0104" H 3400 5500 50  0001 C CNN
+F 0 "#PWR067" H 3400 5500 50  0001 C CNN
 F 1 "GND" H 3405 5577 50  0000 C CNN
 F 2 "" H 3400 5750 50  0001 C CNN
@@
 AR Path="/7D8CCC7A/7D8FC78C" Ref="C27"  Part="1"
 AR Path="/847B579A/7D8FC78C" Ref="C30"  Part="1"
-F 0 "C30" H 2165 2596 50  0000 L CNN
+F 0 "C27" H 2165 2596 50  0000 L CNN
 F 1 "0.1uF" H 2165 2505 50  0000 L CNN
 F 2 "Capacitor_SMD:C_0805_2012Metric_Pad1.18x1.45mm_HandSolder" H 2088 2400 50  0001 C CNN
@@
 AR Path="/7D8CCC7A/7D8FC798" Ref="C28"  Part="1"
 AR Path="/847B579A/7D8FC798" Ref="C31"  Part="1"
-F 0 "C31" H 2615 2946 50  0000 L CNN
+F 0 "C28" H 2615 2946 50  0000 L CNN
 F 1 "0.1uF" H 2615 2855 50  0000 L CNN
 F 2 "Capacitor_SMD:C_0805_2012Metric_Pad1.18x1.45mm_HandSolder" H 2538 2750 50  0001 C CNN
@@
 AR Path="/7D8CCC7A/7D8FC79F" Ref="#PWR065"  Part="1"
 AR Path="/847B579A/7D8FC79F" Ref="#PWR0105"  Part="1"
-F 0 "#PWR0105" H 1450 2500 50  0001 C CNN
+F 0 "#PWR065" H 1450 2500 50  0001 C CNN
 F 1 "GND" H 1455 2577 50  0000 C CNN
 F 2 "" H 1450 2750 50  0001 C CNN
@@
 AR Path="/7D8CCC7A/65D0C082" Ref="J13"  Part="1"
 AR Path="/847B579A/65D0C082" Ref="J23"  Part="1"
-F 0 "J23" H 9221 1696 50  0000 R CNN
+F 0 "J13" H 9221 1696 50  0000 R CNN
 F 1 "AVR-ISP-6" H 9221 1605 50  0000 R CNN
 F 2 "Connector_PinHeader_2.54mm:PinHeader_2x03_P2.54mm_Vertical" V 9300 1650 50  0001 C CNN
@@
 AR Path="/7D8CCC7A/65D67928" Ref="#PWR068"  Part="1"
 AR Path="/847B579A/65D67928" Ref="#PWR0106"  Part="1"
-F 0 "#PWR0106" H 9450 650 50  0001 C CNN
+F 0 "#PWR068" H 9450 650 50  0001 C CNN
 F 1 "+5V" H 9465 973 50  0000 C CNN
 F 2 "" H 9450 800 50  0001 C CNN
@@
 AR Path="/7D8CCC7A/65D7AB96" Ref="#PWR069"  Part="1"
 AR Path="/847B579A/65D7AB96" Ref="#PWR0107"  Part="1"
-F 0 "#PWR0107" H 9450 2150 50  0001 C CNN
+F 0 "#PWR069" H 9450 2150 50  0001 C CNN
 F 1 "GND" H 9455 2227 50  0000 C CNN
 F 2 "" H 9450 2400 50  0001 C CNN
@@
 AR Path="/7D8CCC7A/623C8548" Ref="J14"  Part="1"
 AR Path="/847B579A/623C8548" Ref="J24"  Part="1"
-F 0 "J24" H 9518 2925 50  0000 C CNN
+F 0 "J14" H 9518 2925 50  0000 C CNN
 F 1 "Conn_01x06 (Serial Connector)" H 9518 3016 50  0000 C CNN
 F 2 "Connector_PinHeader_2.54mm:PinHeader_1x06_P2.54mm_Vertical" H 9600 3450 50  0001 C CNN
@@
 AR Path="/7D8CCC7A/65E08A07" Ref="#PWR070"  Part="1"
 AR Path="/847B579A/65E08A07" Ref="#PWR0108"  Part="1"
-F 0 "#PWR0108" H 10100 2600 50  0001 C CNN
+F 0 "#PWR070" H 10100 2600 50  0001 C CNN
 F 1 "+5V" H 10115 2923 50  0000 C CNN
 F 2 "" H 10100 2750 50  0001 C CNN
@@
 AR Path="/7D8CCC7A/65DF3F8A" Ref="#PWR071"  Part="1"
 AR Path="/847B579A/65DF3F8A" Ref="#PWR0109"  Part="1"
-F 0 "#PWR0109" H 10350 4150 50  0001 C CNN
+F 0 "#PWR071" H 10350 4150 50  0001 C CNN
 F 1 "GND" H 10355 4227 50  0000 C CNN
 F 2 "" H 10350 4400 50  0001 C CNN
@@
 AR Path="/7D8CCC7A/65D916C2" Ref="C29"  Part="1"
 AR Path="/847B579A/65D916C2" Ref="C32"  Part="1"
-F 0 "C32" V 9398 4250 50  0000 C CNN
+F 0 "C29" V 9398 4250 50  0000 C CNN
 F 1 "0.1uF" V 9489 4250 50  0000 C CNN
 F 2 "Capacitor_SMD:C_0805_2012Metric_Pad1.18x1.45mm_HandSolder" H 9688 4100 50  0001 C CNN
@@
 AR Path="/7D8CCC7A/7DB0C2C2" Ref="J12"  Part="1"
 AR Path="/847B579A/7DB0C2C2" Ref="J22"  Part="1"
-F 0 "J22" H 7430 5942 50  0000 L CNN
+F 0 "J12" H 7430 5942 50  0000 L CNN
 F 1 "Conn_01x03" H 7430 5851 50  0000 L CNN
 F 2 "Connector_PinHeader_2.54mm:PinHeader_1x03_P2.54mm_Vertical" H 7350 5900 50  0001 C CNN
@@
 AR Path="/7D8CCC7A/8791B6EA" Ref="#PWR0110"  Part="1"
 AR Path="/847B579A/8791B6EA" Ref="#PWR0111"  Part="1"
-F 0 "#PWR0111" H 3500 450 50  0001 C CNN
+F 0 "#PWR0110" H 3500 450 50  0001 C CNN
 F 1 "+5V" H 3515 773 50  0000 C CNN
 F 2 "" H 3500 600 50  0001 C CNN
@@
 $EndComp
 Connection ~ 3500 600
+$Comp
+L Device:R R7
+U 1 1 6197E4D2
+P 4750 6500
+AR Path="/7D8CCC7A/6197E4D2" Ref="R7"  Part="1"
+AR Path="/847B579A/6197E4D2" Ref="R8"  Part="1"
+F 0 "R7" H 4820 6546 50  0000 L CNN
+F 1 "10k" H 4820 6455 50  0000 L CNN
+F 2 "Resistor_SMD:R_0805_2012Metric_Pad1.20x1.40mm_HandSolder" V 4680 6500 50  0001 C CNN
+F 3 "~" H 4750 6500 50  0001 C CNN
+	1    4750 6500
+	1    0    0    -1
+$EndComp
+Wire Wire Line
+	4750 6650 4750 6900
+Wire Wire Line
+	4750 6900 5500 6900
+Text Label 5500 6900 2    50   ~ 0
+~PRG_RESET
+Wire Wire Line
+	4750 6350 4750 5850
+$Comp
+L power:+5V #PWR039
+U 1 1 61981728
+P 4750 5850
+AR Path="/7D8CCC7A/61981728" Ref="#PWR039"  Part="1"
+AR Path="/847B579A/61981728" Ref="#PWR040"  Part="1"
+F 0 "#PWR039" H 4750 5700 50  0001 C CNN
+F 1 "+5V" H 4765 6023 50  0000 C CNN
+F 2 "" H 4750 5850 50  0001 C CNN
+F 3 "" H 4750 5850 50  0001 C CNN
+	1    4750 5850
+	1    0    0    -1
+$EndComp
 $EndSCHEMATC
